Commit message: ROS2 version for the AGV-OTA (ROS Noetic) packages

File: agv_description/urdf/agv.urdf.xacro (robot description, xacro)
@@ -22,9 +22,6 @@
 	<xacro:agv_swivel xyz_caster="-0.37 -0.22 -0.048" rpy_caster="0 0 0" side="back_right"/>
 	<xacro:agv_swivel xyz_caster="-0.37 0.22 -0.048" rpy_caster="0 0 0" side="back_left"/>
-	<!-- Motor plugin -->
 	<xacro:agv_diff_drive />
-	<!-- Joints plugin -->
 	<xacro:agv_joints_state_publisher />
-	<!-- IMU Plugin-->
 	<xacro:agv_imu />
 </robot>

File: agv_description/urdf/agv_base.urdf.xacro (robot description, xacro)
@@ -7,5 +7,5 @@
         <origin xyz="0 0 -0.1625" rpy=" 0 0 0"/>
         <geometry>
-          <mesh filename="package://agv_description/meshes/OTAv07_meshes/OTA-v0.7.stl" scale="0.001 0.001 0.001"/>
+          <mesh filename="file://$(find agv_description)/meshes/OTAv07_meshes/OTA-v0.7.stl" scale="0.001 0.001 0.001"/>
         </geometry>
       </visual>
@@ -13,5 +13,5 @@
         <origin xyz="0 0 -0.075" rpy=" 0 0 0"/>
         <geometry>
-          <!--<mesh filename="package://agv_description/meshes/OTAv07_meshes/OTA-v0.7.stl" scale="0.001 0.001 0.001"/> -->
+          <!--<mesh filename="file://$(find agv_description)/meshes/OTAv07_meshes/OTA-v0.7.stl" scale="0.001 0.001 0.001"/> -->
           <box size="1.02 0.72 0.14"/>
         </geometry>
@@ -22,10 +22,9 @@
       <material value="Gazebo/Orange"/>
     </gazebo>
-    <!-- Laser -->
     <link name="scan_link">
       <visual>
         <origin xyz="0 0 0" rpy="1.570796 0 -1.570796"/>
         <geometry>
-          <mesh filename="package://agv_description/meshes/OTAv07_meshes/S30B-XXXXXX.stl" scale="0.001 0.001 0.001"/>
+          <mesh filename="file://$(find agv_description)/meshes/OTAv07_meshes/S30B-XXXXXX.stl" scale="0.001 0.001 0.001"/>
         </geometry>
       </visual>
@@ -43,44 +42,42 @@
       <axis xyz="0 0 1"/>
     </joint>
+    <!-- Laser -->
     <gazebo reference="scan_link">
-      <material value="Gazebo/DarkGray"/>
-      <sensor type="ray" name="laser_scan">
-      	<tf_prefix></tf_prefix>
-        <pose>0 0 0 0 0 0</pose>
-        <visualize>false</visualize>
-        <update_rate>40</update_rate>
-        <ray>
-          <scan>
-            <horizontal>
-              <samples>720</samples>
-              <resolution>1</resolution>
-              <min_angle>-1.570796</min_angle>	<!-- -2.35619 -->
-              <max_angle>1.570796</max_angle>	<!--  2.35619 -->
-            </horizontal>
-          </scan>
-          <range>
-            <min>0.10</min>
-            <max>30.0</max>
-            <resolution>0.03</resolution>
-          </range>
-          <noise>
-            <type>gaussian</type>
-            <mean>0.0</mean>
-            <stddev>0.01</stddev>
-          </noise>
-        </ray>
-        <plugin name="laser_scan_plugin" filename="libgazebo_ros_laser.so">
-            <topicName>laser</topicName>
-            <frameName>scan_link</frameName>
-            <tf_prefix>/</tf_prefix>
-        </plugin>
+    <material value="Gazebo/DarkGray"/>
+    <sensor name="lidar" type="gpu_lidar">
+         <always_on>true</always_on>
+         <visualize>true</visualize>
+         <pose>0 0 0 0 0 0</pose>
+         <update_rate>40</update_rate>
+         <topic>laser</topic>
+         <gz_frame_id>scan_link</gz_frame_id>
+         <lidar>
+            <scan>
+               <horizontal>
+                  <samples>720</samples>
+                  <update_rate>10</update_rate>
+                  <min_angle>-1.570796</min_angle>
+                  <max_angle>1.570796</max_angle>
+               </horizontal>
+            </scan>
+            <range>
+               <min>0.1</min>
+               <max>30</max>
+               <resolution>0.03</resolution>
+            </range>
+            <noise>
+               <type>gaussian</type>
+               <mean>0.0</mean>
+               <stddev>0.01</stddev>
+            </noise>
+         </lidar>
       </sensor>
-    </gazebo>
+      </gazebo>
     <!-- Zed Camera -->
     <link name="zed_camera">
       <visual>
-          <origin xyz="0 0 0" rpy="0 0 0"/>
+      <origin xyz="0 0 0" rpy="0 0 0"/>
           <geometry>
-            <mesh filename="package://agv_description/meshes/OTAv07_meshes/zed.stl" />
+            <mesh filename="file://$(find agv_description)/meshes/OTAv07_meshes/zed.stl" />
           </geometry>
           <material name="black">
@@ -101,43 +98,37 @@
       <parent link="base_link"/>
       <child link="zed_camera"/>
-      <origin xyz="0.49 0 0.175" rpy="0 0 0" />
+       <origin xyz="0.49 0 0.175" rpy="0 0 0" />
     </joint>
-    <gazebo reference="zed_camera">
-      <sensor type="camera" name="camera">
-        <update_rate>30.0</update_rate>
-        <camera name="head">
-          <horizontal_fov>1.3962634</horizontal_fov>
-          <image>
+  <gazebo reference="zed_camera">
+  <sensor name="camera" type="camera">
+         <always_on>true</always_on>
+         <update_rate>30</update_rate>
+         <visualize>true</visualize>
+         <topic>image_raw</topic>
+         <gz_frame_id>zed_camera</gz_frame_id>
+         <camera name="head">
+          <camera_info_topic>camera_info</camera_info_topic>
+            <horizontal_fov>1.3962634</horizontal_fov>
+            <image>
             <width>640</width>
             <height>480</height>
             <format>R8G8B8</format>
           </image>
-          <clip>
+            <clip>
             <near>0.02</near>
             <far>300</far>
           </clip>
-          <noise>
+            <!-- <optical_frame_id>camera_optical_frame</optical_frame_id> -->
+            <distortion>
+            <k1>0</k1>
+            <k2>0</k2>
+            <k3>0</k3>
+            </distortion>
+             <noise>
             <type>gaussian</type>
-            <!-- Noise is sampled independently per pixel on each frame.
-                That pixel's noise value is added to each of its color
-                channels, which at that point lie in the range [0,1]. -->
             <mean>0.0</mean>
             <stddev>0.007</stddev>
           </noise>
-        </camera>
-        <plugin name="camera_controller" filename="libgazebo_ros_camera.so">
-          <alwaysOn>true</alwaysOn>
-          <updateRate>0.0</updateRate>
-          <cameraName>camera</cameraName>
-          <imageTopicName>image_raw</imageTopicName>
-          <cameraInfoTopicName>camera_info</cameraInfoTopicName>
-          <frameName>zed_camera</frameName>
-          <hackBaseline>0.07</hackBaseline>
-          <distortionK1>0.0</distortionK1>
-          <distortionK2>0.0</distortionK2>
-          <distortionK3>0.0</distortionK3>
-          <distortionT1>0.0</distortionT1>
-          <distortionT2>0.0</distortionT2>
-        </plugin>
+         </camera>
       </sensor>
     </gazebo>

File: agv_description/urdf/agv_caster.urdf.xacro (robot description, xacro)
@@ -7,5 +7,5 @@
         <origin xyz="0 0 0" rpy=" 0 0 0"/>
         <geometry>
-          <mesh filename="package://agv_description/meshes/OTAv07_meshes/SarhosTeker.stl" scale="0.001 0.001 0.001"/>
+          <mesh filename="file://$(find agv_description)/meshes/OTAv07_meshes/SarhosTeker.stl" scale="0.001 0.001 0.001"/>
         </geometry>
       </visual>
@@ -45,4 +45,8 @@
       <child link="caster_wheel_${side}_link"/>
     </joint>
+    <!-- <gazebo reference="caster_wheel_${side}_link">
+    <mu1>0.001</mu1>
+    <mu2>0.001</mu2>
+  </gazebo> -->
   </xacro:macro>
 </robot>

File: agv_description/urdf/agv_ir.urdf.xacro (robot description, xacro)
@@ -11,5 +11,5 @@
 			<origin xyz="0 0 0" rpy="0 0 0"/>
 			<geometry>
-				<mesh filename="package://agv_description/meshes/OTAv07_meshes/FotoelektrikSensor.stl" scale="0.0015 0.0015 0.0015"/>
+				<mesh filename="file://$(find agv_description)/meshes/OTAv07_meshes/FotoelektrikSensor.stl" scale="0.0015 0.0015 0.0015"/>
 			</geometry>
 		</visual>
@@ -27,6 +27,11 @@
 	</joint>
 	<gazebo reference="${link_name}_link">
-		<sensor type="ray" name="${link_name}">
+		<sensor type="gpu_lidar" name="${link_name}">
+		<always_on>1</always_on>
+			<update_rate>4</update_rate>
+			<visualize>true</visualize>
 			<pose>0 0 0 0 0 0</pose>
+			<topic>${link_name}</topic>
+			<frame_id>${link_name}_link</frame_id>
 			<ray>
 				<scan>
@@ -44,15 +49,4 @@
 				</range>
 			</ray>
-			<plugin name="gazebo_ros_range" filename="libgazebo_ros_range.so">
-				<topicName>${link_name}</topicName>
-				<frameName>${link_name}_link</frameName>
-				<frameId>${link_name}_link</frameId>
-				<radiation>ultrasound</radiation>
-				<fov>0.7</fov>
-				<gaussianNoise>0</gaussianNoise>
-			</plugin>
-			<always_on>1</always_on>
-			<update_rate>4</update_rate>
-			<visualize>false</visualize>
 		</sensor>
     </gazebo>

File: agv_description/urdf/agv_plugin.urdf.xacro (robot description, xacro)
@@ -1,70 +1,98 @@
 <?xml version="1.0"?>
 <robot xmlns:xacro="http://ros.org/wiki/xacro">
-  <!-- Joint State Publisher -->
   <xacro:macro name="agv_joints_state_publisher">
   	<gazebo>
-         <plugin name="joint_state_publisher" filename="libgazebo_ros_joint_state_publisher.so">
-            <jointName>caster_front_left_joint,caster_front_right_joint,caster_back_left_joint,caster_back_right_joint,caster_front_left_wheel_joint,caster_front_right_wheel_joint,caster_back_left_wheel_joint,caster_back_right_wheel_joint</jointName>
-            <updateRate>10.0</updateRate>
-            <alwaysOn>true</alwaysOn>
-         </plugin>
+         <plugin filename="gz-sim-joint-state-publisher-system"
+         name="gz::sim::systems::JointStatePublisher">
+         <topic>joint_states</topic>
+         <!-- <joint_name>wheel_right_base</joint_name>
+         <joint_name>wheel_left_base</joint_name> -->
+         <joint_name>caster_front_left_joint</joint_name>
+         <joint_name>caster_front_right_joint</joint_name>
+         <joint_name>caster_back_right_joint</joint_name>
+         <joint_name>caster_back_left_joint</joint_name>
+         <joint_name>caster_front_left_wheel_joint</joint_name>
+         <joint_name>caster_front_right_wheel_joint</joint_name>
+         <joint_name>caster_back_left_wheel_joint</joint_name>
+         <joint_name>caster_back_right_wheel_joint</joint_name>
+         <updateRate>10.0</updateRate>
+      </plugin>
     </gazebo>
   </xacro:macro>
-  <!-- Differential Drive Plugin-->
   <xacro:macro name="agv_diff_drive">
     <gazebo>
-      <plugin name="differential_drive_controller" filename="libgazebo_ros_diff_drive.so">
-        <rosDebugLevel>Debug</rosDebugLevel>
-        <publishWheelTF>false</publishWheelTF>
-        <publishOdomTF>true</publishOdomTF>
-        <publishWheelJointState>true</publishWheelJointState>
-        <alwaysOn>true</alwaysOn>
-        <leftJoint>wheel_right_base</leftJoint>
-        <rightJoint>wheel_left_base</rightJoint>
-        <wheelSeparation>0.60</wheelSeparation>
-        <wheelDiameter>0.20</wheelDiameter>
-        <wheelTorque>20</wheelTorque>
+       <plugin
+         filename="gz-sim-diff-drive-system"
+         name="gz::sim::systems::DiffDrive">
+         <left_joint>wheel_right_base</left_joint>
+         <right_joint>wheel_left_base</right_joint>
+         <wheel_separation>0.60</wheel_separation>
+         <wheel_radius>0.10</wheel_radius>
+         <topic>cmd_vel</topic>
+         <maximum_linear_acceleration>2</maximum_linear_acceleration>
+         <max_velocity>5</max_velocity>
+         <!-- <min_velocity>0</min_velocity> -->
+         <odom_topic>odom</odom_topic>
+         <frame_id>odom</frame_id>
+         <odom_publisher_frequency>30</odom_publisher_frequency>
+         <child_frame_id>base_link</child_frame_id>
+         <tf_topic>/tf</tf_topic>
+         <wheelTorque>20</wheelTorque>
         <wheelAcceleration>1.8</wheelAcceleration>
-        <commandTopic>cmd_vel</commandTopic>
-        <odometryTopic>odom</odometryTopic>
-        <odometryFrame>odom</odometryFrame>
-        <odometrySource>world</odometrySource>
-        <robotBaseFrame>base_link</robotBaseFrame>
-	      <legacyMode>true</legacyMode>
-	      <publishTf>true</publishTf>
         <updateRate>150.0</updateRate>
       </plugin>
     </gazebo>
   </xacro:macro>
-  <!-- IMU Plugin -->
   <xacro:macro name="agv_imu">
-    <gazebo>
-      <plugin name="imu_plugin" filename="libgazebo_ros_imu.so">
-        <alwaysOn>true</alwaysOn>
-        <bodyName>imu_link</bodyName>
-        <frameName>imu_link</frameName>
-        <topicName>imu</topicName>
-        <serviceName>imu_service</serviceName>
-        <gaussianNoise>0.0</gaussianNoise>
-        <updateRate>200</updateRate>
-        <imu>
-          <noise>
-            <type>gaussian</type>
-            <rate>
-              <mean>0.0</mean>
-              <stddev>2e-4</stddev>
-              <bias_mean>0.0000075</bias_mean>
-              <bias_stddev>0.0000008</bias_stddev>
-            </rate>
-            <accel>
-              <mean>0.0</mean>
-              <stddev>1.7e-2</stddev>
-              <bias_mean>0.1</bias_mean>
-              <bias_stddev>0.001</bias_stddev>
-            </accel>
-          </noise>
-        </imu>
-      </plugin>
-    </gazebo>
+  <gazebo reference = "imu_link">
+    <sensor name="imu" type="imu">
+    <always_on>true</always_on>
+    <update_rate>200</update_rate>
+    <gz_frame_id>imu_link</gz_frame_id>
+    <topic>imu</topic>
+    <imu>
+     <angular_velocity>
+            <x>
+              <noise type="gaussian">
+                <mean>0.0</mean>
+                <stddev>2e-4</stddev>
+              </noise>
+            </x>
+            <y>
+              <noise type="gaussian">
+                <mean>0.0</mean>
+                <stddev>2e-4</stddev>
+              </noise>
+            </y>
+            <z>
+              <noise type="gaussian">
+                <mean>0.0</mean>
+                <stddev>2e-4</stddev>
+              </noise>
+            </z>
+          </angular_velocity>
+          <linear_acceleration>
+            <x>
+              <noise type="gaussian">
+                <mean>0.0</mean>
+                <stddev>1.7e-2</stddev>
+              </noise>
+            </x>
+            <y>
+              <noise type="gaussian">
+                <mean>0.0</mean>
+                <stddev>1.7e-2</stddev>
+              </noise>
+            </y>
+            <z>
+              <noise type="gaussian">
+                <mean>0.0</mean>
+                <stddev>1.7e-2</stddev>
+              </noise>
+            </z>
+          </linear_acceleration>
+    </imu>
+  </sensor>
+  </gazebo>
   </xacro:macro>
 </robot>

File: agv_description/urdf/agv_wheel.urdf.xacro (robot description, xacro)
@@ -6,5 +6,5 @@
         <origin xyz="0 0 0" rpy=" 0 0 1.570796"/>
         <geometry>
-          <mesh filename="package://agv_description/meshes/OTAv07_meshes/AnaTeker.stl" scale="0.001 0.001 0.001"/>
+          <mesh filename="file://$(find agv_description)/meshes/OTAv07_meshes/AnaTeker.stl" scale="0.001 0.001 0.001"/>
         </geometry>
       </visual>
@@ -24,4 +24,8 @@
     </joint>
     <gazebo reference="wheel_${side}_link">
+    <!-- <mu1>1.5</mu1>
+  <mu2>1.5</mu2>
+  <kp>1000000</kp>
+  <kd>10</kd> -->
       <material value="Gazebo/Green"/>
     </gazebo>
